File: shiftBoard/shiftBoard.kicad_pcb (KiCad board)
At the start: 2 copper layers, 88 x 93 mm, 54 parts, among them J1 Screw_Terminal_01x02, J10 Screw_Terminal_01x02, J11 Screw_Terminal_01x02, J12 Screw_Terminal_01x02, J2 Screw_Terminal_01x02, J3 Screw_Terminal_01x02, J4 Screw_Terminal_01x02, J5 Screw_Terminal_01x02, J6 Screw_Terminal_01x02, J7 Screw_Terminal_01x02, J8 Screw_Terminal_01x02, J9 Screw_Terminal_01x02, Q1 AO3400A, Q2 AO3400A, Q3 AO3400A, Q4 AO3400A, Q5 AO3400A, Q6 AO3400A, Q7 AO3400A, Q8 AO3400A, U2 74HC595

Commit message: nameing and pcb mounting holes
Parts:
- added H1: MountingHole, MountingHole:MountingHole_3.2mm_M3, F.Cu at (212.5, 108.5)
- added H2: MountingHole, MountingHole:MountingHole_3.2mm_M3, F.Cu at (212.5, 53.5)
- added H3: MountingHole, MountingHole:MountingHole_3.2mm_M3, F.Cu at (171.5, 50.0)
- added H4: MountingHole, MountingHole:MountingHole_3.2mm_M3, F.Cu at (171.5, 106.5)
- turned R14 to 180 degrees
Connections:
- net Net-(J2-Pin_1) renamed /push
- net Net-(J2-Pin_2) renamed /shift
- net Net-(J3-Pin_2) renamed /Bit
- net Net-(U2-QA) renamed /Q1
- net Net-(U2-QB) renamed /Q2
- net Net-(U2-QC) renamed /Q3
- net Net-(U2-QD) renamed /Q4
- net Net-(U2-QE) renamed /Q5
- net Net-(U2-QF) renamed /Q6
- net Net-(U2-QG) renamed /Q7
- net Net-(U2-QH) renamed /Q8
Routing:
- net /VCC: track 53.1 -> 58.7 mm

Commit message: bypass fixed
Parts:
- moved C1 14.3 mm to (192.5, 70.0), turned to 0 degrees
Connections:
- C1 pad 2: /VCC -> /GND
Routing:
- net /VCC: track 58.7 -> 45.5 mm
- net /GND: track 278.4 -> 280.7 mm
Changed lines of the file:
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@@
 	(footprint "Capacitor_SMD:C_1206_3216Metric_Pad1.33x1.80mm_HandSolder"
 		(layer "F.Cu")
-		(at 183.9375 58.5 -90)
+		(at 192.5 70)
 		(descr "Capacitor SMD 1206 (3216 Metric), square (rectangular) end terminal, IPC-7351 nominal with elongated pad for handsoldering. (Body size source: IPC-SM-782 page 76, https://www.pcb-3d.com/wordpress/wp-content/uploads/ipc-sm-782a_amendment_1_and_2.pdf), generated with kicad-footprint-generator")
 		(tags "capacitor handsolder")
 		(property "Reference" "C1"
-			(at 0 -1.85 90)
+			(at 0 -1.85 0)
 			(layer "F.SilkS")
 			(effects
@@
 		)
 		(property "Value" "100nF"
-			(at 0 1.85 90)
+			(at 0 1.85 0)
 			(layer "F.Fab")
 			(effects
@@
 		)
 		(property "Datasheet" "~"
-			(at 0 0 90)
+			(at 0 0 0)
 			(layer "F.Fab")
 			(hide yes)
@@
 		)
 		(property "Description" "Unpolarized capacitor"
-			(at 0 0 90)
+			(at 0 0 0)
 			(layer "F.Fab")
 			(hide yes)
@@
 		(attr smd)
 		(fp_line
-			(start -0.711252 0.91)
-			(end 0.711252 0.91)
+			(start -0.711252 -0.91)
+			(end 0.711252 -0.91)
 			(stroke
 				(width 0.12)
@@
 		)
 		(fp_line
-			(start -0.711252 -0.91)
-			(end 0.711252 -0.91)
+			(start -0.711252 0.91)
+			(end 0.711252 0.91)
 			(stroke
 				(width 0.12)
@@
 		)
 		(fp_text user "${REFERENCE}"
-			(at 0 0 90)
+			(at 0 0 0)
 			(layer "F.Fab")
 			(effects
@@
 		)
 		(pad "1" smd roundrect
-			(at -1.5625 0 270)
+			(at -1.5625 0)
 			(size 1.325 1.8)
 			(layers "F.Cu" "F.Mask" "F.Paste")
@@
 		)
 		(pad "2" smd roundrect
-			(at 1.5625 0 270)
+			(at 1.5625 0)
 			(size 1.325 1.8)
 			(layers "F.Cu" "F.Mask" "F.Paste")
 			(roundrect_rratio 0.188679)
-			(net 2 "/VCC")
+			(net 1 "/GND")
 			(pintype "passive")
 		)
@@
 	)
 	(segment
+		(start 194.0625 72.6675)
+		(end 194 72.73)
+		(width 0.2)
+		(layer "F.Cu")
+		(net 1)
+	)
+	(segment
 		(start 233 47)
 		(end 232 48)
@@
 	)
 	(segment
+		(start 194.0625 70.5)
+		(end 194.0625 72.6675)
+		(width 0.2)
+		(layer "F.Cu")
+		(net 1)
+	)
+	(segment
 		(start 231.99 81.01)
 		(end 232 81)
@@
 	)
 	(segment
-		(start 183.9375 60.0625)
-		(end 179.0625 60.0625)
-		(width 0.2)
-		(layer "F.Cu")
-		(net 2)
-	)
-	(segment
-		(start 179.5625 60.0625)
-		(end 179.5 60)
-		(width 0.2)
-		(layer "F.Cu")
-		(net 2)
-	)
-	(segment
 		(start 193 80)
 		(end 193 75)
@@
 	)
 	(segment
-		(start 179 59.5)
-		(end 179.5 60)
-		(width 0.2)
-		(layer "F.Cu")
-		(net 2)
-	)
-	(segment
 		(start 171.6175 58.0525)
 		(end 178.0525 58.0525)
@@
 	)
 	(segment
-		(start 179.1675 56.9375)
-		(end 178.0525 58.0525)
+		(start 191.5 71.0625)
+		(end 191.5 74)
 		(width 0.2)
 		(layer "F.Cu")
@@
 	)
 	(segment
-		(start 183.9375 56.9375)
-		(end 179.1675 56.9375)
+		(start 191.5 74)
+		(end 190 74)
 		(width 0.2)
 		(layer "F.Cu")
@@
 	)
 	(segment
-		(start 179.0625 60.0625)
-		(end 179 60)
+		(start 190.9375 70.5)
+		(end 191.5 71.0625)
 		(width 0.2)
 		(layer "F.Cu")
@@
 	)
 	(segment
-		(start 179.5 60)
-		(end 179 60)
-		(width 0.2)
-		(layer "F.Cu")
-		(net 2)
-	)
-	(segment
-		(start 183.9375 60.0625)
-		(end 179.5625 60.0625)
-		(width 0.2)
-		(layer "F.Cu")
-		(net 2)
-	)
-	(segment
 		(start 192 74)
-		(end 190 74)
+		(end 191.5 74)
 		(width 0.2)
 		(layer "F.Cu")

Commit message: holes and final print
Parts:
- moved H1 20.2 mm to (199.5, 124.0)
- moved H4 17.8 mm to (168.0, 124.0)
- moved H2 16.7 mm to (199.5, 43.0)
- moved H3 7.83 mm to (168.0, 43.0)
Routing:
- net /GND: track 280.7 -> 281.3 mm, vias 10 -> 11

Commit message: :(
Connections:
- J2 pad 1: /push -> /shift
- J2 pad 2: /shift -> /latch
- U2 pad 11: /push -> /shift
- U2 pad 12: /shift -> /latch
Routing:
- net /push: track 20.5 -> 0.00 mm
- net /latch: track 0.00 -> 19.0 mm
- net /shift: track 19.0 -> 20.5 mm
Changed lines of the file:
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@@
 	(net 37 "Net-(D15-A)")
 	(net 38 "Net-(D16-A)")
-	(net 39 "/push")
+	(net 39 "/latch")
 	(footprint "Diode_THT:D_DO-41_SOD81_P10.16mm_Horizontal"
 		(layer "F.Cu")
@@
 			(size 1.7018 0.5334)
 			(layers "F.Cu" "F.Mask" "F.Paste")
-			(net 39 "/push")
+			(net 3 "/shift")
 			(pinfunction "SRCLK")
 			(pintype "input")
@@
 			(size 1.7018 0.5334)
 			(layers "F.Cu" "F.Mask" "F.Paste")
-			(net 3 "/shift")
+			(net 39 "/latch")
 			(pinfunction "RCLK")
 			(pintype "input")
@@
 			(remove_unused_layers no)
 			(roundrect_rratio 0.096154)
-			(net 39 "/push")
+			(net 3 "/shift")
 			(pinfunction "Pin_1")
 			(pintype "passive")
@@
 			(layers "*.Cu" "*.Mask")
 			(remove_unused_layers no)
-			(net 3 "/shift")
+			(net 39 "/latch")
 			(pinfunction "Pin_2")
 			(pintype "passive")
@@
 	)
 	(segment
-		(start 179.1025 75.1025)
-		(end 171.6175 75.1025)
+		(start 181.27 75.27)
+		(end 176.1025 70.1025)
 		(width 0.5)
 		(layer "F.Cu")
@@
 	)
 	(segment
-		(start 180.54 76.54)
-		(end 179.1025 75.1025)
+		(start 190 75.27)
+		(end 181.27 75.27)
 		(width 0.5)
 		(layer "F.Cu")
@@
 	)
 	(segment
-		(start 190 76.54)
-		(end 180.54 76.54)
+		(start 176.1025 70.1025)
+		(end 171.6175 70.1025)
 		(width 0.5)
 		(layer "F.Cu")
@@
 	)
 	(segment
-		(start 181.27 75.27)
-		(end 176.1025 70.1025)
+		(start 179.1025 75.1025)
+		(end 171.6175 75.1025)
 		(width 0.5)
 		(layer "F.Cu")
@@
 	)
 	(segment
-		(start 190 75.27)
-		(end 181.27 75.27)
+		(start 180.54 76.54)
+		(end 179.1025 75.1025)
 		(width 0.5)
 		(layer "F.Cu")
@@
 	)
 	(segment
-		(start 176.1025 70.1025)
-		(end 171.6175 70.1025)
+		(start 190 76.54)
+		(end 180.54 76.54)
 		(width 0.5)
 		(layer "F.Cu")
